File: hardware/modules/vga-v2/output.sch (KiCad schematic (older format))
At the start: 12 parts, among them J401 DB15_Female_HighDensity_Mount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, U401 SN74LVC541A

Commit message: VGA Module V2 Production Files
Various changes, including: Smaller VGA connector, fix soldermask
Parts:
- J401: footprint Connector_Dsub:DSUB-15-HD_Female_Horizontal_P2.29x1.98mm_EdgePinOffset8.35mm_Housed_MountingHolesOffset10.89mm -> Connector_Dsub:DSUB-15-HD_Female_Horizontal_P2.29x1.98mm_EdgePinOffset3.03mm_Housed_MountingHolesOffset4.94mm
Changed lines of the file:
@@
 F 0 "J401" H 7950 4817 50  0000 C CNN
 F 1 "DB15_Female_HighDensity_MountingHoles" H 7950 4726 50  0000 C CNN
-F 2 "Connector_Dsub:DSUB-15-HD_Female_Horizontal_P2.29x1.98mm_EdgePinOffset8.35mm_Housed_MountingHolesOffset10.89mm" H 7000 4350 50  0001 C CNN
+F 2 "Connector_Dsub:DSUB-15-HD_Female_Horizontal_P2.29x1.98mm_EdgePinOffset3.03mm_Housed_MountingHolesOffset4.94mm" H 7000 4350 50  0001 C CNN
 F 3 " ~" H 7000 4350 50  0001 C CNN
 	1    7950 3950
